Commit message: mppi based planner works now. made ur5 robot to be bigger. tested with multiple init + goal configs.

File: urdf/bed_0.urdf (robot description, URDF)
Before this commit: robot cube.urdf, 1 links, 0 joints
Links:
- link baseLink: geometry collision box size=0.8 1.9 0.3; visual box size=0.8 2.0 0.4

Commit message: pcd is fixed (now based on meshes/collision/visual data), attaching grasped object control points to robot control points is added, doing more collision check (sometimes works sometime collides)

File: urdf/bed_0.urdf (robot description, URDF)
Before this commit: robot cube.urdf, 1 links, 0 joints
Links:
- link baseLink: geometry collision box size=0.5 1.6 0.3; visual box size=0.6 1.6 0.4

Commit message: planning and control method completed. collision check and constraints are both considered. currently adding in generating grasps (this needs to be completed).

File: urdf/bed_0.urdf (robot description, URDF)
Before this commit: robot cube.urdf, 1 links, 0 joints
Links:
- link baseLink: geometry collision box size=0.5 1.7 0.3; visual box size=0.6 1.7 0.4

File: urdf/humanoid_simplified_rev_scaled.urdf (robot description, URDF)
Before this commit: robot dumpUrdf, 7 links, 6 joints
Links:
- link right_elbow: geometry collision capsule length=0.118800 radius=0.035200
- link right_shoulder: geometry collision capsule length=0.158400 radius=0.039600
- link right_wrist: geometry collision sphere radius=0.035200
Joints:
- joint right_elbow: origin xyz=0.000000 -1.099152 0.000000 rpy=0 0 0 -> xyz=0.000000 -0.241813 0.000000 rpy=0 0 0
- joint right_wrist: origin xyz=0.000000 -1.035788 0.000000 rpy=0 0 0 -> xyz=0.000000 -0.227873 0.000000 rpy=0 0 0
- joint shoulder_roll: origin xyz=-0.096200 0.974000 0.732440 rpy=0 0 0 -> xyz=-0.021164 0.214280 0.161137 rpy=0 0 0

File: urdf/humanoid_with_rev.urdf (robot description, URDF)
Before this commit: robot dumpUrdf, 19 links, 18 joints
Links:
- link right_elbow: geometry collision capsule length=0.540000 radius=0.140000
- link right_shoulder: geometry collision capsule length=0.620000 radius=0.180000
- link right_wrist: geometry collision sphere radius=0.140000
